File: PCBs/MelodicChimes/MelodicChimes/MelodicChimes.sch (KiCad schematic (older format))
At the start: 14 parts

Commit message: PCB work.
Parts:
- removed U? (x4): DRV8838, Package_SON:WSON-8-1EP_2x2mm_P0.5mm_EP0.9x1.6mm, symbol Driver_Motor:DRV8838
- added U1, U10, U12, U4: TMC2208_SILENTSTEPSTICK, MODULE_TMC2208_SILENTSTEPSTICK, symbol stepper-drivers:TMC2208_SILENTSTEPSTICK
- gave numbers to parts that had none: 10
Other:
- moved on the sheet: U11, U13, U8, U9
